File: batteryController/batteryControllerCncPcb/batteryControllerCncPcb.kicad_sch (KiCad schematic)
At the start: 15 parts, among them J1 Conn_01x02_Male, J2 Screw_Terminal_01x02, J3 Conn_01x04_Male, J4 Conn_01x04_Male, J5 Conn_01x04_Male, J6 USB_A, U1 ATtiny13V-10P, U2 L7806CV, U3 L78L05_TO92

Commit message: remade basically the entire thing
Parts:
- R2, R4: value R -> 2k
- R3, R5: value R -> 680
Changed lines of the file:
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@@
       (effects (font (size 1.27 1.27)) (justify left))
     )
-    (property "Value" "R" (id 1) (at 164.338 94.4122 0)
+    (property "Value" "680" (id 1) (at 164.338 94.4122 0)
       (effects (font (size 1.27 1.27)) (justify left))
     )
@@
       (effects (font (size 1.27 1.27)) (justify left))
     )
-    (property "Value" "R" (id 1) (at 150.368 94.4122 0)
+    (property "Value" "680" (id 1) (at 150.368 94.4122 0)
       (effects (font (size 1.27 1.27)) (justify left))
     )
@@
       (effects (font (size 1.27 1.27)) (justify left))
     )
-    (property "Value" "R" (id 1) (at 144.018 94.4122 0)
+    (property "Value" "2k" (id 1) (at 144.018 94.4122 0)
       (effects (font (size 1.27 1.27)) (justify left))
     )
@@
       (effects (font (size 1.27 1.27)) (justify left))
     )
-    (property "Value" "R" (id 1) (at 157.988 94.4122 0)
+    (property "Value" "2k" (id 1) (at 157.988 94.4122 0)
       (effects (font (size 1.27 1.27)) (justify left))
     )
@@
     )
     (path "/efbd3197-cbc9-408a-a2b5-e8292a952aae"
-      (reference "R2") (unit 1) (value "R") (footprint "Resistor_THT:R_Axial_DIN0207_L6.3mm_D2.5mm_P7.62mm_Horizontal")
+      (reference "R2") (unit 1) (value "2k") (footprint "Resistor_THT:R_Axial_DIN0207_L6.3mm_D2.5mm_P7.62mm_Horizontal")
     )
     (path "/4fd71c9f-fda7-44dc-a730-71f9a293687a"
-      (reference "R3") (unit 1) (value "R") (footprint "Resistor_THT:R_Axial_DIN0207_L6.3mm_D2.5mm_P7.62mm_Horizontal")
+      (reference "R3") (unit 1) (value "680") (footprint "Resistor_THT:R_Axial_DIN0207_L6.3mm_D2.5mm_P7.62mm_Horizontal")
     )
     (path "/f6c853d4-bbcd-4b7b-9a09-2cb0aa558725"
-      (reference "R4") (unit 1) (value "R") (footprint "Resistor_THT:R_Axial_DIN0207_L6.3mm_D2.5mm_P7.62mm_Horizontal")
+      (reference "R4") (unit 1) (value "2k") (footprint "Resistor_THT:R_Axial_DIN0207_L6.3mm_D2.5mm_P7.62mm_Horizontal")
     )
     (path "/136ccffd-861c-43d7-9c0d-f960a50fef7f"
-      (reference "R5") (unit 1) (value "R") (footprint "Resistor_THT:R_Axial_DIN0207_L6.3mm_D2.5mm_P7.62mm_Horizontal")
+      (reference "R5") (unit 1) (value "680") (footprint "Resistor_THT:R_Axial_DIN0207_L6.3mm_D2.5mm_P7.62mm_Horizontal")
     )
     (path "/074bd178-4b8d-4443-a5fb-cfcbc87a942c"
